Commit message: New calibration

File: assets/lighthouse/robot.urdf (robot description, URDF)
Before this commit: robot onshape, 3 links, 2 joints
Links:
- link arrow_1_0: geometry collision mesh filename=package://arrow.stl; visual mesh filename=package://arrow.stl
- link arrow_1_1: geometry collision mesh filename=package://box.stl; visual mesh filename=package://box.stl
