Commit message: Changing the trackers frame to X front led, Z top

File: assets/tracker.urdf (robot description, URDF)
Before this commit: robot tracker, 1 links, 0 joints
Links:
- link trackerLink: geometry collision mesh filename=tracker_x_led.stl scale=0.001 0.001 0.001; visual mesh filename=tracker_x_led.stl scale=0.001 0.001 0.001

Commit message: Offset commented

File: assets/tracker.urdf (robot description, URDF)
Before this commit: robot tracker, 1 links, 0 joints
Links:
- link trackerLink: geometry collision mesh filename=vr_tracker_vive_x_led.stl scale=1 1 1; visual mesh filename=vr_tracker_vive_x_led.stl scale=1 1 1
