Commit message: Adding tables

File: assets/field/robot.urdf (robot description, URDF)
Before this commit: robot onshape, 9 links, 8 joints
Links:
- added link field_1_10, mass 0.000000; collision mesh filename=package://penaltyally.stl; visual mesh filename=package://penaltyally.stl
- added link field_1_11, mass 0.000000; collision mesh filename=package://lines.stl; visual mesh filename=package://lines.stl
- added link field_1_8, mass 0.000000; collision mesh filename=package://goalsopponentback.stl; visual mesh filename=package://goalsopponentback.stl
- added link field_1_9, mass 0.000000; collision mesh filename=package://field.stl; visual mesh filename=package://field.stl
- link field_1_0: geometry collision mesh filename=package://table4.stl; visual mesh filename=package://table4.stl
- link field_1_1: geometry collision mesh filename=package://penaltyopponent.stl; visual mesh filename=package://penaltyopponent.stl
- link field_1_2: geometry collision mesh filename=package://goalsally.stl; visual mesh filename=package://goalsally.stl
- link field_1_3: geometry collision mesh filename=package://table2.stl; visual mesh filename=package://table2.stl
- link field_1_4: geometry collision mesh filename=package://table3.stl; visual mesh filename=package://table3.stl
- link field_1_5: geometry collision mesh filename=package://goalsopponent.stl; visual mesh filename=package://goalsopponent.stl
- link field_1_6: geometry collision mesh filename=package://table.stl; visual mesh filename=package://table.stl
- link field_1_7: geometry collision mesh filename=package://goalsallyback.stl; visual mesh filename=package://goalsallyback.stl
Joints:
- added joint field_1_field_1_10_fixing: type fixed, parent field_1, child field_1_10, origin xyz=0.000000 0.000000 0.000000 rpy=0.000000 -0.000000 0.000000, axis 0 0 0
- added joint field_1_field_1_11_fixing: type fixed, parent field_1, child field_1_11, origin xyz=0.000000 0.000000 0.000000 rpy=0.000000 -0.000000 0.000000, axis 0 0 0
- added joint field_1_field_1_8_fixing: type fixed, parent field_1, child field_1_8, origin xyz=0.000000 0.000000 0.000000 rpy=0.000000 -0.000000 0.000000, axis 0 0 0
- added joint field_1_field_1_9_fixing: type fixed, parent field_1, child field_1_9, origin xyz=0.000000 0.000000 0.000000 rpy=0.000000 -0.000000 0.000000, axis 0 0 0

Commit message: Field update

File: assets/field/robot.urdf (robot description, URDF)
Before this commit: robot onshape, 13 links, 12 joints
Links:
- removed link field_1_0
- removed link field_1_1
- removed link field_1_10
- removed link field_1_11
- removed link field_1_2
- removed link field_1_3
- removed link field_1_4
- removed link field_1_5
- removed link field_1_6
- removed link field_1_7
- removed link field_1_8
- removed link field_1_9
- added link field, mass 0; collision mesh filename=package:///field.stl; collision mesh filename=package:///goalsally.stl
- added link field_10, mass 0; visual mesh filename=package:///field.stl
- added link field_11, mass 0; visual mesh filename=package:///penaltyally.stl
- added link field_12, mass 0; visual mesh filename=package:///lines.stl
- added link field_2, mass 0; visual mesh filename=package:///penaltyopponent.stl
- added link field_3, mass 0; visual mesh filename=package:///goalsally.stl
- added link field_4, mass 0; visual mesh filename=package:///table2.stl
- added link field_5, mass 0; visual mesh filename=package:///table3.stl
- added link field_6, mass 0; visual mesh filename=package:///goalsopponent.stl
- added link field_7, mass 0; visual mesh filename=package:///table.stl
- added link field_8, mass 0; visual mesh filename=package:///goalsallyback.stl
- added link field_9, mass 0; visual mesh filename=package:///goalsopponentback.stl
- link field_1: geometry visual mesh filename=package:///table4.stl
Joints:
- removed joint field_1_field_1_0_fixing
- removed joint field_1_field_1_10_fixing
- removed joint field_1_field_1_11_fixing
- removed joint field_1_field_1_1_fixing
- removed joint field_1_field_1_2_fixing
- removed joint field_1_field_1_3_fixing
- removed joint field_1_field_1_4_fixing
- removed joint field_1_field_1_5_fixing
- removed joint field_1_field_1_6_fixing
- removed joint field_1_field_1_7_fixing
- removed joint field_1_field_1_8_fixing
- removed joint field_1_field_1_9_fixing
- added joint field_10_fixing: type fixed, parent field, child field_10, origin xyz=0 0 0 rpy=0 -0 0, axis 0 0 1, limit effort=1 velocity=20
- added joint field_11_fixing: type fixed, parent field, child field_11, origin xyz=0 0 0 rpy=0 -0 0, axis 0 0 1, limit effort=1 velocity=20
- added joint field_12_fixing: type fixed, parent field, child field_12, origin xyz=0 0 0 rpy=0 -0 0, axis 0 0 1, limit effort=1 velocity=20
- added joint field_1_fixing: type fixed, parent field, child field_1, origin xyz=0 0 0 rpy=0 -0 0, axis 0 0 1, limit effort=1 velocity=20
- added joint field_2_fixing: type fixed, parent field, child field_2, origin xyz=0 0 0 rpy=0 -0 0, axis 0 0 1, limit effort=1 velocity=20
- added joint field_3_fixing: type fixed, parent field, child field_3, origin xyz=0 0 0 rpy=0 -0 0, axis 0 0 1, limit effort=1 velocity=20
- added joint field_4_fixing: type fixed, parent field, child field_4, origin xyz=0 0 0 rpy=0 -0 0, axis 0 0 1, limit effort=1 velocity=20
- added joint field_5_fixing: type fixed, parent field, child field_5, origin xyz=0 0 0 rpy=0 -0 0, axis 0 0 1, limit effort=1 velocity=20
- added joint field_6_fixing: type fixed, parent field, child field_6, origin xyz=0 0 0 rpy=0 -0 0, axis 0 0 1, limit effort=1 velocity=20
- added joint field_7_fixing: type fixed, parent field, child field_7, origin xyz=0 0 0 rpy=0 -0 0, axis 0 0 1, limit effort=1 velocity=20
- added joint field_8_fixing: type fixed, parent field, child field_8, origin xyz=0 0 0 rpy=0 -0 0, axis 0 0 1, limit effort=1 velocity=20
- added joint field_9_fixing: type fixed, parent field, child field_9, origin xyz=0 0 0 rpy=0 -0 0, axis 0 0 1, limit effort=1 velocity=20
